File: Hardware/RC thing_G/RC thing.kicad_pcb (KiCad board)
At the start: 2 copper layers, 100.1 x 80 mm, 53 parts, among them J1 Conn_01x04, P1 USB_C_Plug_USB2.0, SW2 SW_Push, SW3 SW_Push, SW302 TL3342F160QG_TR, SW4 SW_Push, U1 MCP73831-2-OT, U101 NRF24L01_Breakout, U2 RP2040, U3 W25Q128JVS, U401 TPS62170DSG, Y3 Crystal_GND24_Small

Commit message: the G-ening
Parts:
- removed C18, C20: 4.7u, Capacitor_THT:CP_Radial_D6.3mm_P2.50mm
- removed C409: 100n, Capacitor_SMD:C_0603_1608Metric_Pad1.08x0.95mm_HandSolder
- removed J1: Conn_01x04, Connector_PinHeader_2.54mm:PinHeader_1x04_P2.54mm_Vertical
- removed R410: 100k, Resistor_SMD:R_0603_1608Metric_Pad0.98x0.95mm_HandSolder
- removed R411: 360k, Resistor_SMD:R_0603_1608Metric_Pad0.98x0.95mm_HandSolder
- removed RV1, RV2: 4.7k, Connector_JST:JST_PH_B3B-PH-K_1x03_P2.00mm_Vertical
- removed SW302: TL3342F160QG_TR, Button_Switch_SMD:SW_SPST_TL3342
- removed U101: NRF24L01_Breakout, Connector_PinHeader_2.54mm:PinHeader_2x04_P2.54mm_Vertical
- added ?: , , F.Cu at (140.1, 72.8)
- added ?: , , F.Cu at (140.1, 75.3)
- added ?: , , F.Cu at (141.4, 75.3)
- added ?: , , F.Cu at (140.1, 74.0)
- added ?: , , F.Cu at (138.8, 75.3)
- added ?: , , F.Cu at (138.8, 74.0)
- added ?: , , F.Cu at (141.4, 72.8)
- added ?: , , F.Cu at (141.4, 74.0)
- added ?: , , F.Cu at (138.8, 72.8)
- added C30: 100n, Capacitor_SMD:C_0603_1608Metric_Pad1.08x0.95mm_HandSolder, B.Cu at (128.1, 67.2)
- added C402: 4.7u, Capacitor_SMD:C_0805_2012Metric_Pad1.18x1.45mm_HandSolder, B.Cu at (123.3, 58.5)
- added C403: 4.7u, Capacitor_SMD:C_0805_2012Metric_Pad1.18x1.45mm_HandSolder, B.Cu at (122.0, 48.4)
- added C403: 4.7u, Capacitor_SMD:C_0805_2012Metric_Pad1.18x1.45mm_HandSolder, B.Cu at (125.3, 48.3)
- added J2: Conn_01x04, Connector_PinHeader_2.54mm:PinHeader_1x04_P2.54mm_Vertical, B.Cu at (160.2, 68.7)
- added R1: 10k, Capacitor_SMD:C_0603_1608Metric_Pad1.08x0.95mm_HandSolder, B.Cu at (135.3, 88.5)
- added R25: 100k, Resistor_SMD:R_0603_1608Metric_Pad0.98x0.95mm_HandSolder, B.Cu at (124.5, 67.1)
- added R26: 360k, Resistor_SMD:R_0603_1608Metric_Pad0.98x0.95mm_HandSolder, B.Cu at (126.3, 67.1)
- added RV3: 4.7k, Connector_PinHeader_2.54mm:PinHeader_1x03_P2.54mm_Vertical, B.Cu at (127.3, 75.0)
- added RV4: 4.7k, Connector_PinHeader_2.54mm:PinHeader_1x03_P2.54mm_Vertical, B.Cu at (127.3, 70.8)
- added SW1: TL3342F160QG_TR, Main_PCB:SW_TL3342F160QG_TR, B.Cu at (128.8, 89.5)
- added SW5: TL3342F160QG_TR, Main_PCB:SW_TL3342F160QG_TR, B.Cu at (149.6, 46.8)
- added U102: NRF24L01_Breakout, Connector_PinHeader_2.54mm:PinHeader_2x04_P2.54mm_Vertical, B.Cu at (125.0, 81.0)
- BT1, C401, SW2, SW3, SW4: moved to B.Cu
- C13: value 100n -> 100nx3
- C9: value 100n -> 100nx2
- moved H3 158.1 mm to (164.2, 89.9)
- moved H2 148.6 mm to (164.2, 45.1)
- moved H4 111.0 mm to (115.9, 89.9)
- moved H1 102.4 mm to (115.9, 45.1)
- moved BT1 61.4 mm to (117.1, 63.0), turned to 90 degrees
- moved C401 54.4 mm to (122.3, 62.0), turned to 90 degrees
- moved C11 17.8 mm to (126.4, 78.0), turned to 180 degrees
- moved SW4 15.7 mm to (155.1, 84.0), turned to 90 degrees
- moved SW2 14.2 mm to (155.1, 74.8), turned to 90 degrees
- moved SW3 7.74 mm to (155.1, 79.4), turned to 90 degrees
- moved R404 5.48 mm to (132.9, 62.6)
- moved C12 5.34 mm to (145.6, 77.2), turned to -90 degrees
- moved R405 5.20 mm to (132.9, 60.5)
- moved U1 5.05 mm to (125.3, 54.2)
- moved L402 4.83 mm to (129.5, 62.6), turned to 90 degrees
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Connections:
- C404 pad 1: +3.3V -> +3V3
- L402 pad 2: +3.3V -> +3V3
- R403 pad 2: +3.3V -> +3V3
- R404 pad 2: +3.3V -> +3V3
- SW2 pad 2: /Button1 -> /RP2040/Button1
- SW3 pad 2: /Button2 -> /RP2040/Button2
- SW4 pad 2: /Button3 -> /RP2040/Button3
- U1 pad 1: /BMS and power/Charge_status -> /RP2040/Charge_status
- U2 pad 14: /RP2040/Charge_status -> /RP2040/GPIO11
- U2 pad 2: /RP2040/GPIO0 -> /RP2040/SDA
- U2 pad 26: /RP2040/RUN -> Net-(U2-RUN)
- U2 pad 27: /RP2040/GPIO16 -> /RP2040/MISO
- U2 pad 29: /RP2040/GPIO18 -> /RP2040/SCK
- U2 pad 3: /RP2040/GPIO1 -> /RP2040/SCL
- U2 pad 30: /RP2040/GPIO19 -> /RP2040/MOSI
- U2 pad 31: /RP2040/GPIO20 -> /RP2040/CE
- U2 pad 32: /RP2040/GPIO21 -> /RP2040/CSN
- U2 pad 34: /RP2040/GPIO22 -> /RP2040/Charge_status
- U2 pad 38: /RP2040/GPIO26_ADC0 -> /RP2040/AnaStk_1
- U2 pad 39: /RP2040/GPIO27_ADC1 -> /RP2040/AnaStk_2
- U2 pad 40: /RP2040/GPIO28_ADC2 -> /RP2040/Battery_voltage_level
- U2 pad 6: /RP2040/GPIO4 -> /RP2040/Button1
- U2 pad 7: /RP2040/GPIO5 -> /RP2040/Button2
- U2 pad 8: /RP2040/GPIO6 -> /RP2040/Button3
- U401 pad 6: +3.3V -> +3V3
Routing:
- net +3V3: track 46.1 -> 130.4 mm, vias 3 -> 8
- net GND: track 37.9 -> 79.2 mm, vias 15 -> 22
- net /RP2040/Charge_status: track 0.00 -> 25.2 mm, vias 0 -> 2
- net /RP2040/CSN: track 0.00 -> 16.4 mm
- net Net-(U2-RUN): track 0.00 -> 15.9 mm
- net /RP2040/Battery_voltage_level: track 0.00 -> 15.3 mm
- net /RP2040/Button3: track 0.00 -> 15.2 mm
- net +3.3V: track 14.3 -> 0.00 mm, vias 1 -> 0
- net VBAT: track 6.33 -> 20.6 mm
- net /RP2040/MOSI: track 0.00 -> 13.4 mm
- net /RP2040/SCL: track 0.00 -> 13.0 mm
- net /RP2040/AnaStk_1: track 0.00 -> 12.7 mm
- net /RP2040/AnaStk_2: track 0.00 -> 12.6 mm
- net /RP2040/CE: track 0.00 -> 11.3 mm
- net /RP2040/Button2: track 0.00 -> 11.2 mm
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- added copper zone on B.Cu, net GND
- added copper zone on F.Cu, net GND
Other:
- board size 100.1 x 80 mm -> 56.4 x 52.8 mm
- board text added: "->"
- board text added: "IN ORDER"
- board text added: "x2"
- board text added: "|"

Commit message: cleanup 2
Parts:
- added D2: D_0603_1608Metric_Pad1.05x0.95mm_HandSolder, Diode_SMD:D_0603_1608Metric_Pad1.05x0.95mm_HandSolder, B.Cu at (133.1, 55.5)
- added R1: R_0603_1608Metric_Pad0.98x0.95mm_HandSolder, Resistor_SMD:R_0603_1608Metric_Pad0.98x0.95mm_HandSolder, B.Cu at (133.1, 57.5)
Routing:
- net /RP2040/Charge_status: track 25.2 -> 30.5 mm
- net +3V3: track 130.4 -> 134.0 mm
- net (no net): track 0.00 -> 2.00 mm

Commit message: current state of Rc
Parts:
- removed C402, C403 (x2): 4.7u, Capacitor_SMD:C_0805_2012Metric_Pad1.18x1.45mm_HandSolder
- removed P1: USB_C_Plug_USB2.0, Connector_USB:USB_C_Receptacle_Molex_105450-0101
- added C18: 4.7u, Capacitor_SMD:C_0805_2012Metric_Pad1.18x1.45mm_HandSolder, B.Cu at (123.0, 58.0)
- added C20: 4.7u, Capacitor_SMD:C_0805_2012Metric_Pad1.18x1.45mm_HandSolder, B.Cu at (125.5, 48.0)
- added J2: 2171790001, rctg:2171790001_MOL, B.Cu at (139.0, 44.0)
- added R6: 5.1k, Resistor_SMD:R_0603_1608Metric_Pad0.98x0.95mm_HandSolder, B.Cu at (137.0, 52.9)
- added SW1: Bat_switch, Connector_JST:JST_PH_B2B-PH-K_1x02_P2.00mm_Vertical, B.Cu at (115.5, 62.5)
- BT1: footprint Connector_JST:JST_PH_B3B-PH-K_1x03_P2.00mm_Vertical -> Connector_JST:JST_PH_B2B-PH-K_1x02_P2.00mm_Vertical
- C13: value 100nx3 -> 100n
- D2: value D_0603_1608Metric_Pad1.05x0.95mm_HandSolder -> LED
- R1: value R_0603_1608Metric_Pad0.98x0.95mm_HandSolder -> 240
- moved BT1 8.15 mm to (115.5, 55.0), turned to -90 degrees
- moved R3 4.84 mm to (141.5, 50.9)
- moved C16 0.55 mm to (134.5, 52.5)
- moved R5 0.31 mm to (140.0, 59.5)
- moved D2 0.25 mm to (132.9, 55.5), turned to 0 degrees
- moved R4 0.24 mm to (138.0, 59.4)
- moved U1 0.20 mm to (125.5, 54.4)
- moved R1 0.18 mm to (132.9, 57.5)
Connections:
- BT1 pad 1: VBAT -> Net-(BT1-+)
- D2 pad 1: (no net) -> /BMS and power/Charge_status
- D2 pad 2: /RP2040/Charge_status -> /BMS and power/D2_in
- R1 pad 2: (no net) -> /BMS and power/D2_in
- U1 pad 1: /RP2040/Charge_status -> /BMS and power/Charge_status
- U2 pad 2: /RP2040/SDA -> /RP2040/GPIO0
- U2 pad 26: Net-(U2-RUN) -> /RP2040/RUN
- U2 pad 27: /RP2040/MISO -> /RP2040/GPIO16
- U2 pad 29: /RP2040/SCK -> /RP2040/GPIO18
- U2 pad 3: /RP2040/SCL -> /RP2040/GPIO1
- U2 pad 30: /RP2040/MOSI -> /RP2040/GPIO19
- U2 pad 31: /RP2040/CE -> /RP2040/GPIO20
- U2 pad 32: /RP2040/CSN -> /RP2040/GPIO21
- U2 pad 34: /RP2040/Charge_status -> /RP2040/GPIO22
- U2 pad 38: /RP2040/AnaStk_1 -> /RP2040/GPIO26_ADC0
- U2 pad 39: /RP2040/AnaStk_2 -> /RP2040/GPIO27_ADC1
- U2 pad 40: /RP2040/Battery_voltage_level -> /RP2040/GPIO28_ADC2
- U2 pad 6: /RP2040/Button1 -> /RP2040/GPIO4
- U2 pad 7: /RP2040/Button2 -> /RP2040/GPIO5
- U2 pad 8: /RP2040/Button3 -> /RP2040/GPIO6
Routing:
- net /RP2040/Charge_status: track 30.5 -> 0.00 mm, vias 2 -> 0
- net (no net): track 2.00 -> 30.2 mm
- net GND: track 79.2 -> 62.3 mm, vias 22 -> 20
- net Net-(BT1-+): track 0.00 -> 9.57 mm
- net Net-(J2-CC1): track 0.00 -> 5.13 mm
- net Net-(J2-DP1): track 10.3 -> 15.4 mm
- net Net-(J2-DN1): track 10.3 -> 13.8 mm
- net Net-(D1-A): track 13.5 -> 16.5 mm
- net VUSB: track 13.9 -> 11.0 mm
- net VBAT: track 20.6 -> 22.9 mm
- net /BMS and power/D2_in: track 0.00 -> 2.03 mm
- net Net-(J2-CC2): track 3.52 -> 3.01 mm
- net /RP2040/GPIO11: vias 0 -> 2
