File: Hardware/RC thing_G/RC thing.kicad_sch (KiCad schematic)
At the start: 11 parts, among them J1 Conn_01x04, SW2 SW_Push, SW3 SW_Push, SW4 SW_Push, U101 NRF24L01_Breakout

Commit message: cleanup
Connections:
- net GPIO3 is gone; now on net GPIO4: SW2.2
- net GPIO4: no longer SW3.2
- net GPIO5: now also SW3.2; no longer SW4.2
- net GPIO12 renamed GPIO0
- net GPIO13 renamed GPIO1
- net GPIO7 renamed GPIO20
- net GPIO8 renamed GPIO21
- new net GPIO6: SW4.2
Changed lines of the file:
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@@
 		)
 	)
-	(hierarchical_label "GPIO7"
+	(hierarchical_label "GPIO20"
 		(shape tri_state)
 		(at 46.99 27.94 180)
@@
 		)
 	)
-	(hierarchical_label "GPIO5"
+	(hierarchical_label "GPIO6"
 		(shape tri_state)
 		(at 46.99 55.88 180)
@@
 		)
 	)
-	(hierarchical_label "GPIO13"
+	(hierarchical_label "GPIO1"
 		(shape tri_state)
 		(at 46.99 62.23 180)
@@
 		)
 	)
-	(hierarchical_label "GPIO11"
+	(hierarchical_label "GPIO22"
 		(shape tri_state)
 		(at 46.99 68.58 180)
@@
 		)
 	)
-	(hierarchical_label "GPIO12"
+	(hierarchical_label "GPIO0"
 		(shape tri_state)
 		(at 46.99 59.69 180)
@@
 		)
 	)
-	(hierarchical_label "GPIO8"
+	(hierarchical_label "GPIO21"
 		(shape tri_state)
 		(at 46.99 30.48 180)
@@
 		)
 	)
-	(hierarchical_label "GPIO3"
+	(hierarchical_label "GPIO4"
 		(shape tri_state)
 		(at 46.99 50.8 180)
@@
 		)
 	)
-	(hierarchical_label "GPIO4"
+	(hierarchical_label "GPIO5"
 		(shape tri_state)
 		(at 46.99 53.34 180)

Commit message: cleanup 2
Connections:
- net +3.3V: no longer U101.2 (VCC)
- net +3V3: now also U101.2 (VCC)
Changed lines of the file:
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@@
 			)
 		)
-		(property "Value" "+3.3V"
-			(at 254 30.48 0)
+		(property "Value" "+3V3"
+			(at 256.54 34.2899 0)
 			(effects
 				(font
 					(size 1.27 1.27)
 				)
+				(justify left)
 			)
 		)

Commit message: current state of Rc
Connections:
- net +3.3V is gone; now on net +3V3: J1.2 (Pin_2)
- net GPIO26 renamed GPIO26_ADC0
- net GPIO27 renamed GPIO27_ADC1
Changed lines of the file:
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@@
+	(wire
+		(pts
+			(xy 50.8 68.58) (xy 50.8 80.01)
+		)
+		(stroke
+			(width 0)
+			(type default)
+		)
+	)
+	(wire
+		(pts
+			(xy 54.61 66.04) (xy 54.61 82.55)
+		)
+		(stroke
+			(width 0)
+			(type default)
+		)
+	)
+	(wire
+		(pts
+			(xy 46.99 30.48) (xy 57.15 30.48)
+		)
+		(stroke
+			(width 0)
+			(type default)
+		)
+	)
+	(wire
+		(pts
+			(xy 46.99 55.88) (xy 57.15 55.88)
+		)
+		(stroke
+			(width 0)
+			(type default)
+		)
+	)
 	(wire
 		(pts
 			(xy 90.17 71.12) (xy 95.25 71.12)
-		)
-		(stroke
-			(width 0)
-			(type default)
-		)
-	)
-	(wire
-		(pts
-			(xy 50.8 68.58) (xy 50.8 80.01)
-		)
-		(stroke
-			(width 0)
-			(type default)
-		)
-	)
-	(wire
-		(pts
-			(xy 54.61 66.04) (xy 54.61 82.55)
-		)
-		(stroke
-			(width 0)
-			(type default)
-		)
-	)
-	(wire
-		(pts
-			(xy 46.99 30.48) (xy 57.15 30.48)
-		)
-		(stroke
-			(width 0)
-			(type default)
-		)
-	)
-	(wire
-		(pts
-			(xy 46.99 55.88) (xy 57.15 55.88)
 		)
 		(stroke
@@
 		)
 	)
+	(label "Button1"
+		(at 95.25 77.47 0)
+		(effects
+			(font
+				(size 1.27 1.27)
+			)
+			(justify left bottom)
+		)
+	)
 	(label "MOSI"
 		(at 57.15 38.1 0)
@@
 	(label "Button1"
 		(at 57.15 50.8 0)
-		(effects
-			(font
-				(size 1.27 1.27)
-			)
-			(justify left bottom)
-		)
-	)
-	(label "Button1"
-		(at 95.25 77.47 0)
 		(effects
 			(font
@@
 		)
 	)
+	(hierarchical_label "GPIO1"
+		(shape bidirectional)
+		(at 46.99 62.23 180)
+		(effects
+			(font
+				(size 1.27 1.27)
+			)
+			(justify right)
+		)
+	)
 	(hierarchical_label "GPIO20"
 		(shape tri_state)
@@
 		)
 	)
-	(hierarchical_label "GPIO1"
-		(shape tri_state)
-		(at 46.99 62.23 180)
-		(effects
-			(font
-				(size 1.27 1.27)
-			)
-			(justify right)
-		)
-	)
 	(hierarchical_label "GPIO16"
 		(shape tri_state)
@@
 		)
 	)
-	(hierarchical_label "GPIO0"
-		(shape tri_state)
-		(at 46.99 59.69 180)
-		(effects
-			(font
-				(size 1.27 1.27)
-			)
-			(justify right)
-		)
-	)
 	(hierarchical_label "GPIO21"
 		(shape tri_state)
@@
 		)
 	)
-	(hierarchical_label "GPIO26"
+	(hierarchical_label "GPIO26_ADC0"
 		(shape tri_state)
 		(at 46.99 44.45 180)
@@
 		)
 	)
-	(hierarchical_label "GPIO27"
+	(hierarchical_label "GPIO27_ADC1"
 		(shape tri_state)
 		(at 46.99 46.99 180)
@@
 		)
 	)
+	(hierarchical_label "GPIO0"
+		(shape bidirectional)
+		(at 46.99 59.69 180)
+		(effects
+			(font
+				(size 1.27 1.27)
+			)
+			(justify right)
+		)
+	)
 	(hierarchical_label "GPIO5"
 		(shape tri_state)
@@
 		)
 	)
-	(hierarchical_label "GPIO28"
+	(hierarchical_label "GPIO28_ADC2"
 		(shape tri_state)
 		(at 46.99 66.04 180)
@@
 			)
 		)
-		(property "Value" "+3.3V"
+		(property "Value" "+3V3"
 			(at 152.4 30.48 0)
 			(effects
