File: Hardware/RC thing_G/bms.kicad_sch (KiCad schematic)
At the start: 15 parts, among them U1 MCP73831-2-OT, U401 TPS62170DSG

Commit message: cleanup 2
Parts:
- added D2: LED, Diode_SMD:D_0603_1608Metric_Pad1.05x0.95mm_HandSolder, symbol Device:LED
- added R1: 240, Resistor_SMD:R_0603_1608Metric_Pad0.98x0.95mm_HandSolder, symbol Device:R
Connections:
- net Charge_status: now also D2.1 (K)
- net +3.3V renamed +3V3
- net +3V3: now also R1.1
- new net D2_in: D2.2 (A), R1.2
Other:
- moved on the sheet: C409, R410, R411

Commit message: current state of Rc
Parts:
- added SW1: Bat_switch, Connector_JST:JST_PH_B2B-PH-K_1x02_P2.00mm_Vertical, symbol Switch:SW_SPST
- BT1: footprint Connector_JST:JST_PH_B3B-PH-K_1x03_P2.00mm_Vertical -> Connector_JST:JST_PH_B2B-PH-K_1x02_P2.00mm_Vertical
- C18, C20: footprint Capacitor_THT:CP_Radial_D6.3mm_P2.50mm -> Capacitor_SMD:C_0805_2012Metric_Pad1.18x1.45mm_HandSolder
Connections:
- net VBAT: now also SW1.2 (B); no longer BT1.1 (+)
- new net: BT1.1 (+), SW1.1 (A)
Other:
- moved on the sheet: BT1
Changed lines of the file:
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@@
+	)
+	(junction
+		(at 96.52 40.64)
+		(diameter 0)
+		(color 0 0 0 0)
 	)
 	(junction
@@
 	(junction
 		(at 190.5 39.37)
-		(diameter 0)
-		(color 0 0 0 0)
-	)
-	(junction
-		(at 96.52 40.64)
 		(diameter 0)
 		(color 0 0 0 0)
@@
 			)
 		)
-		(property "Footprint" "Capacitor_THT:CP_Radial_D6.3mm_P2.50mm"
+		(property "Footprint" "Capacitor_SMD:C_0805_2012Metric_Pad1.18x1.45mm_HandSolder"
 			(at 46.99 26.9748 0)
 			(effects
@@
 	)
 	(symbol
+		(lib_id "Switch:SW_SPST")
+		(at 96.52 45.72 90)
+		(unit 1)
+		(exclude_from_sim no)
+		(in_bom yes)
+		(on_board yes)
+		(dnp no)
+		(fields_autoplaced yes)
+		(property "Reference" "SW1"
+			(at 97.79 44.4499 90)
+			(effects
+				(font
+					(size 1.27 1.27)
+				)
+				(justify right)
+			)
+		)
+		(property "Value" "Bat_switch"
+			(at 97.79 46.9899 90)
+			(effects
+				(font
+					(size 1.27 1.27)
+				)
+				(justify right)
+			)
+		)
+		(property "Footprint" "Connector_JST:JST_PH_B2B-PH-K_1x02_P2.00mm_Vertical"
+			(at 96.52 45.72 0)
+			(effects
+				(font
+					(size 1.27 1.27)
+				)
+				(hide yes)
+			)
+		)
+		(property "Datasheet" "~"
+			(at 96.52 45.72 0)
+			(effects
+				(font
+					(size 1.27 1.27)
+				)
+				(hide yes)
+			)
+		)
+		(property "Description" "Single Pole Single Throw (SPST) switch"
+			(at 96.52 45.72 0)
+			(effects
+				(font
+					(size 1.27 1.27)
+				)
+				(hide yes)
+			)
+		)
+		(pin "1"
+		)
+		(pin "2"
+		)
+		(instances
+			(project ""
+				(path "/5c54a15d-2138-46dc-867e-29c9270be5e0/87ff3aa1-14e4-4935-92da-05f81d408638"
+					(reference "SW1")
+					(unit 1)
+				)
+			)
+		)
+	)
+	(symbol
 		(lib_id "Device:R")
 		(at 176.53 58.42 180)
@@
 			)
 		)
-		(property "Footprint" "Capacitor_THT:CP_Radial_D6.3mm_P2.50mm"
+		(property "Footprint" "Capacitor_SMD:C_0805_2012Metric_Pad1.18x1.45mm_HandSolder"
 			(at 77.1652 48.26 0)
 			(effects
@@
 	(symbol
 		(lib_id "power:GND")
-		(at 96.52 48.26 0)
+		(at 96.52 58.42 0)
 		(unit 1)
 		(exclude_from_sim no)
@@
 		(fields_autoplaced yes)
 		(property "Reference" "#PWR04"
-			(at 96.52 54.61 0)
+			(at 96.52 64.77 0)
 			(effects
 				(font
@@
 		)
 		(property "Value" "GND"
-			(at 96.52 53.34 0)
+			(at 96.52 63.5 0)
 			(effects
 				(font
@@
 		)
 		(property "Footprint" ""
-			(at 96.52 48.26 0)
+			(at 96.52 58.42 0)
 			(effects
 				(font
@@
 		)
 		(property "Datasheet" ""
-			(at 96.52 48.26 0)
+			(at 96.52 58.42 0)
 			(effects
 				(font
@@
 		)
 		(property "Description" "Power symbol creates a global label with name \"GND\" , ground"
-			(at 96.52 48.26 0)
+			(at 96.52 58.42 0)
 			(effects
 				(font
@@
 	(symbol
 		(lib_id "Device:Battery_Cell")
-		(at 96.52 45.72 0)
+		(at 96.52 55.88 0)
 		(unit 1)
 		(exclude_from_sim no)
@@
 		(fields_autoplaced yes)
 		(property "Reference" "BT1"
-			(at 100.33 42.6084 0)
+			(at 100.33 52.7684 0)
 			(effects
 				(font
@@
 		)
 		(property "Value" "Battery_Cell"
-			(at 100.33 45.1484 0)
+			(at 100.33 55.3084 0)
 			(effects
 				(font
@@
 			)
 		)
-		(property "Footprint" "Connector_JST:JST_PH_B3B-PH-K_1x03_P2.00mm_Vertical"
-			(at 96.52 44.196 90)
+		(property "Footprint" "Connector_JST:JST_PH_B2B-PH-K_1x02_P2.00mm_Vertical"
+			(at 96.52 54.356 90)
 			(effects
 				(font
@@
 		)
 		(property "Datasheet" "~"
-			(at 96.52 44.196 90)
+			(at 96.52 54.356 90)
 			(effects
 				(font
@@
 		)
 		(property "Description" "Single-cell battery"
-			(at 96.52 45.72 0)
-			(effects
-				(font
+			(at 96.52 55.88 0)
+			(effects
+				(font
