File: Hardware/RC thing_G/rp2040.kicad_sch (KiCad schematic)
At the start: 26 parts, among them P1 USB_C_Plug_USB2.0, SW302 TL3342F160QG_TR, U2 RP2040, U3 W25Q128JVS, Y3 Crystal_GND24_Small

Commit message: current state of Rc
Parts:
- removed P1: USB_C_Plug_USB2.0, Connector_USB:USB_C_Receptacle_Molex_105450-0101, symbol Connector:USB_C_Plug_USB2.0
- added J2: 2171790001, rctg:2171790001_MOL, symbol MainPCB_Sym_lib:2171790001
- added R6: 5.1k, Resistor_SMD:R_0603_1608Metric_Pad0.98x0.95mm_HandSolder, symbol Device:R
Connections:
- net GND: now also J2.A1/B12 (GND), J2.B1/A12 (GND), R6.2
- net at C16.1, D1.2 (A): now also J2.A4/B9 (VBUS), J2.B4/A9 (VBUS)
- net at R4.1: now also J2.A7 (DN1), J2.B7 (DN2)
- net at R5.1: now also J2.A6 (DP1), J2.B6 (DP2)
- net at R3.1: now also J2.B5 (CC2)
- net Charge_status renamed GPIO11
- new net: J2.A5 (CC1), R6.1
- no-connect marks 1 -> 2
Other:
- moved on the sheet: C16, D1, R3
