File: Hardware/ESC and BMS/ESC_BMS/SPROJ3EE_ESC_BMS.kicad_pcb (KiCad board)
At the start: 4 copper layers, 100 x 40 mm, 100 parts, among them J301 SW IN, J302 SW OUT, J401 1mm2_connector, J402 1mm2_connector, J403 1mm2_connector, J404 JST_8PH_2mm, J405 JST_3PH_2mm, J406 1mm2_connector, J407 1mm2_connector, J408 1mm2_connector, J409 1mm2_connector, J410 Barrel_Jack_Switch, Q201 SiR696DP, Q202 SiR696DP, Q203 SiR696DP, Q204 SiR696DP, Q205 SiR696DP, Q206 SiR696DP, Q301 SQJQ131EL, Q303 FDV304P, Q304 PMV20XNEA, Q305 SQJQ131EL, Q306 SQJQ131EL, U201 74AUC2G08, U202 74AUC2G08, U203 SN74LVC1G00DBV, U204 SN74LVC1G00DBV, U205 IR2301, U206 IR2301, U207 74AUC2G08, U208 SN74LVC1G00DBV, U209 TL331, U210 IR2301, U301 BQ2057W, U302 BQ2969

Commit message: Small adjustments
Routing:
- net (no net): track 0.00 -> 24.7 mm
- net /1. ESC/CLS: track 24.1 -> 20.2 mm, vias 2 -> 0
- net Net-(D202-K): track 5.53 -> 8.96 mm
- net GND: track 0.70 -> 3.05 mm, vias 132 -> 137
- net +3.3V: track 102.1 -> 103.5 mm
- net /1. ESC/BLS: track 30.1 -> 31.1 mm, vias 3 -> 1
- net /1. ESC/BHS: track 23.0 -> 22.5 mm, vias 1 -> 0
- net /1. ESC/CNAND: track 11.1 -> 11.4 mm, vias 2 -> 0
- net /1. ESC/CHS: track 36.3 -> 36.6 mm, vias 4 -> 0
- net Net-(U206-HO): track 7.79 -> 7.64 mm, vias 2 -> 0
Other:
- board text added: "JLCJLCJLCJLC"
