File: Hardware/ESC and BMS/ESC_BMS/SPROJ3EE_ESC_BMS.kicad_pcb (KiCad board)
At the start: 4 copper layers, 100 x 40 mm, 100 parts, among them J301 SW IN, J302 SW OUT, J401 1mm2_connector, J402 1mm2_connector, J403 1mm2_connector, J404 JST_8PH_2mm, J405 JST_3PH_2mm, J406 1mm2_connector, J407 1mm2_connector, J408 1mm2_connector, J409 1mm2_connector, J410 Barrel_Jack_Switch, Q201 SiR696DP, Q202 SiR696DP, Q203 SiR696DP, Q204 SiR696DP, Q205 SiR696DP, Q206 SiR696DP, Q301 SQJQ131EL, Q303 FDV304P, Q304 PMV20XNEA, Q305 SQJQ131EL, Q306 SQJQ131EL, U201 74AUC2G08, U202 74AUC2G08, U203 SN74LVC1G00DBV, U204 SN74LVC1G00DBV, U205 IR2301, U206 IR2301, U207 74AUC2G08, U208 SN74LVC1G00DBV, U209 TL331, U210 IR2301, U301 BQ2057W, U302 BQ2969

Commit message: Final touches
Routing:
- net (no net): track 24.7 -> 0.00 mm
Changed lines of the file:
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@@
 			(outputformat 1)
 			(mirror no)
-			(drillshape 1)
+			(drillshape 0)
 			(scaleselection 1)
-			(outputdirectory "")
+			(outputdirectory "../../../../../GerberSPROJ/ESCBMS/")
 		)
 	)
@@
 	)
 	(segment
-		(start 193.463733 109.7)
-		(end 193.2226 109.902335)
-		(width 0.2)
-		(layer "F.Cu")
-		(net 0)
-	)
-	(segment
-		(start 203.7 109.7)
-		(end 193.463733 109.7)
-		(width 0.2)
-		(layer "F.Cu")
-		(net 0)
-	)
-	(segment
-		(start 213.7 119.7)
-		(end 203.7 109.7)
-		(width 0.2)
-		(layer "F.Cu")
-		(net 0)
-	)
-	(segment
