File: Hardware/RC thing/RC thing.kicad_pcb (KiCad board)
At the start: 4 copper layers, 58.1 x 54 mm, 70 parts, among them J1 Conn_01x04, J2 2171790001, SW1 Bat_switch, SW2 SW_Push, SW3 SW_Push, SW4 SW_Push, SW5 TL3342F160QG_TR, SW8 TL3342F160QG_TR, U1 MCP73831-2-OT, U101 NRF24L01_Breakout, U2 RP2040, U3 W25Q128JVS, U401 TPS62170DSG, X1 Crystal_GND24_Small

Commit message: Final touches
Parts:
- renumbered C5 to C1, C13 to C10, C14 to C11, C15 to C12, C1 to C13, C16 to C14, C20 to C15, C18 to C16, C31 to C17, C32 to C18, C33 to C19, C6 to C2, C4 to C3, C2 to C4, C3 to C5, C8 to C6, C10 to C7, C11 to C8, C12 to C9, L2 to L1, R9 to R1, R8 to R10, R2 to R11, R1 to R12, R35 to R13, R37 to R14, R36 to R15, R39 to R16, R38 to R17, R7 to R2, R11 to R3, R12 to R4, R6 to R5, R4 to R6, R5 to R7, R3 to R8, R10 to R9, SW2 to SW1, SW3 to SW2, SW4 to SW3, SW5 to SW4, SW8 to SW5, SW1 to SW6, U101 to U1, U1 to U4, U401 to U5
Other:
- board text added: "JLCJLCJLCJLC"
