File: Hardware/RC thing/RC thing.kicad_sch (KiCad schematic)
At the start: 11 parts, among them J1 Conn_01x04, SW2 SW_Push, SW3 SW_Push, SW4 SW_Push, U101 NRF24L01_Breakout

Commit message: Final touches
Parts:
- renumbered SW2 to SW1, SW3 to SW2, SW4 to SW3, U101 to U1
Changed lines of the file:
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@@
 		(dnp no)
 		(fields_autoplaced yes)
-		(property "Reference" "#PWR029"
+		(property "Reference" "#PWR08"
 			(at 157.48 26.67 0)
 			(effects
@@
 			(project ""
 				(path "/5c54a15d-2138-46dc-867e-29c9270be5e0"
-					(reference "#PWR029")
+					(reference "#PWR08")
 					(unit 1)
 				)
@@
 		(dnp no)
 		(fields_autoplaced yes)
-		(property "Reference" "#PWR028"
+		(property "Reference" "#PWR03"
 			(at 93.98 49.53 0)
 			(effects
@@
 			(project ""
 				(path "/5c54a15d-2138-46dc-867e-29c9270be5e0"
-					(reference "#PWR028")
+					(reference "#PWR03")
 					(unit 1)
 				)
@@
 		(dnp no)
 		(fields_autoplaced yes)
-		(property "Reference" "#PWR032"
+		(property "Reference" "#PWR07"
 			(at 152.4 39.37 0)
 			(effects
@@
 			(project ""
 				(path "/5c54a15d-2138-46dc-867e-29c9270be5e0"
-					(reference "#PWR032")
+					(reference "#PWR07")
 					(unit 1)
 				)
@@
 		(dnp no)
 		(fields_autoplaced yes)
-		(property "Reference" "SW2"
+		(property "Reference" "SW1"
 			(at 85.09 63.5 0)
 			(effects
@@
 			(project ""
 				(path "/5c54a15d-2138-46dc-867e-29c9270be5e0"
-					(reference "SW2")
+					(reference "SW1")
 					(unit 1)
 				)
@@
 		(dnp no)
 		(fields_autoplaced yes)
-		(property "Reference" "SW4"
+		(property "Reference" "SW3"
 			(at 140.97 63.5 0)
 			(effects
@@
 			(project "RC thing"
 				(path "/5c54a15d-2138-46dc-867e-29c9270be5e0"
-					(reference "SW4")
+					(reference "SW3")
 					(unit 1)
 				)
@@
 		(on_board yes)
 		(dnp no)
-		(property "Reference" "U101"
+		(property "Reference" "U1"
 			(at 243.84 49.5299 0)
 			(effects
@@
 			(project "RC thing"
 				(path "/5c54a15d-2138-46dc-867e-29c9270be5e0"
-					(reference "U101")
+					(reference "U1")
 					(unit 1)
 				)
@@
 		(on_board yes)
 		(dnp no)
-		(property "Reference" "#PWR042"
+		(property "Reference" "#PWR010"
 			(at 254 72.39 0)
 			(effects
@@
 			(project "RC thing"
 				(path "/5c54a15d-2138-46dc-867e-29c9270be5e0"
-					(reference "#PWR042")
+					(reference "#PWR010")
 					(unit 1)
 				)
@@
 		(dnp no)
 		(fields_autoplaced yes)
-		(property "Reference" "#PWR030"
+		(property "Reference" "#PWR01"
 			(at 80.01 81.28 0)
 			(effects
@@
 			(project "RC thing"
 				(path "/5c54a15d-2138-46dc-867e-29c9270be5e0"
-					(reference "#PWR030")
+					(reference "#PWR01")
 					(unit 1)
 				)
@@
 		(dnp no)
 		(fields_autoplaced yes)
-		(property "Reference" "#PWR031"
+		(property "Reference" "#PWR04"
 			(at 107.95 81.28 0)
 			(effects
@@
 			(project "RC thing"
 				(path "/5c54a15d-2138-46dc-867e-29c9270be5e0"
-					(reference "#PWR031")
+					(reference "#PWR04")
 					(unit 1)
 				)
@@
 		(dnp no)
 		(fields_autoplaced yes)
-		(property "Reference" "#PWR026"
+		(property "Reference" "#PWR02"
 			(at 93.98 35.56 0)
 			(effects
@@
 			(project ""
 				(path "/5c54a15d-2138-46dc-867e-29c9270be5e0"
-					(reference "#PWR026")
+					(reference "#PWR02")
 					(unit 1)
 				)
@@
 		(dnp no)
 		(fields_autoplaced yes)
-		(property "Reference" "#PWR033"
+		(property "Reference" "#PWR06"
 			(at 135.89 81.28 0)
 			(effects
@@
 			(project "RC thing"
 				(path "/5c54a15d-2138-46dc-867e-29c9270be5e0"
-					(reference "#PWR033")
+					(reference "#PWR06")
 					(unit 1)
 				)
@@
 		(dnp no)
 		(fields_autoplaced yes)
-		(property "Reference" "SW3"
+		(property "Reference" "SW2"
 			(at 113.03 63.5 0)
 			(effects
@@
 			(project ""
 				(path "/5c54a15d-2138-46dc-867e-29c9270be5e0"
-					(reference "SW3")
+					(reference "SW2")
 					(unit 1)
 				)
@@
 		(dnp no)
 		(fields_autoplaced yes)
-		(property "Reference" "#PWR043"
+		(property "Reference" "#PWR09"
 			(at 254 39.37 0)
 			(effects
@@
 			(project "RC thing"
 				(path "/5c54a15d-2138-46dc-867e-29c9270be5e0"
-					(reference "#PWR043")
+					(reference "#PWR09")
 					(unit 1)
 				)
@@
 		(dnp no)
 		(fields_autoplaced yes)
-		(property "Reference" "#PWR027"
+		(property "Reference" "#PWR05"
 			(at 121.92 49.53 0)
 			(effects
@@
 			(project ""
 				(path "/5c54a15d-2138-46dc-867e-29c9270be5e0"
-					(reference "#PWR027")
-					(unit 1)
-				)
+					(reference "#PWR05")
+					(unit 1)
+				)
