File: Hardware/RC thing/rp2040.kicad_sch (KiCad schematic)
At the start: 30 parts, among them P1 USB_C_Plug_USB2.0, SW1 Reset button, SW2 TL3342F160QG_TR, U5 RP2040, U6 W25Q128JVS, Y1 12Mhz

Commit message: RC thing schematic 70% done
Parts:
- removed C23: 100n, Capacitor_SMD:C_0603_1608Metric_Pad1.08x0.95mm_HandSolder, symbol Device:C
- removed C24, C25: 27pF, Capacitor_SMD:C_0603_1608Metric_Pad1.08x0.95mm_HandSolder, symbol Device:C
- removed H1, H2, H3, H4: MountingHole, MountingHole:MountingHole_2.7mm_M2.5, symbol Mechanical:MountingHole
- removed R12: 5.1k, symbol Device:R
- removed R13, R14: 27, symbol Device:R
- removed SW1: Reset button, symbol Switch:SW_Push
- removed U6: W25Q128JVS, Package_SO:SOIC-8_5.23x5.23mm_P1.27mm, symbol Memory_Flash:W25Q128JVS
- added C17: 100n, Capacitor_SMD:C_0603_1608Metric_Pad1.08x0.95mm_HandSolder, symbol Device:C
- added C3: 10u, Capacitor_SMD:C_0603_1608Metric_Pad1.08x0.95mm_HandSolder, symbol Device:C
- added C7, C8: 27pF, Capacitor_SMD:C_0603_1608Metric_Pad1.08x0.95mm_HandSolder, symbol Device:C
- added D1: MSS1P3L-M3/89A, Diode_SMD:Vishay_SMPA, symbol Device:D_Schottky
- added R3: 5.1k, Resistor_SMD:R_0603_1608Metric_Pad0.98x0.95mm_HandSolder, symbol Device:R
- added R4, R5: 27, Resistor_SMD:R_0603_1608Metric_Pad0.98x0.95mm_HandSolder, symbol Device:R
- added U3: W25Q128JVS, Package_SO:SOIC-8_5.23x5.23mm_P1.27mm, symbol Memory_Flash:W25Q128JVS
- P1: footprint (none) -> Connector_USB:USB_C_Receptacle_Molex_105450-0101
- R6: renamed from R16; value 820 -> 820R
- renumbered C22 to C10, C15 to C11, C16 to C12, C17 to C13, C18 to C14, C19 to C15, C20 to C16, C12 to C4, C13 to C5, C21 to C6, C14 to C9, R17 to R7, R15 to R8, SW2 to SW1, U5 to U2
Connections:
- net +3V3: now also C17.1, U3.8 (VCC)
- net GND: now also C17.2, C3.2, C7.2, C8.2, R3.2, U3.4 (GND)
- net QSPI_SCLK: now also U3.6 (CLK)
- net QSPI_SD0: now also U3.5 (DI(IO0))
- net QSPI_SD1: now also U3.2 (DO(IO1))
- net QSPI_SD2: now also U3.3 (IO2)
- net QSPI_SD3: now also U3.7 (IO3)
- net QSPI_SS: now also U3.1 (~{CS})
- net XIN: now also C7.1; no longer R6.1, U2.21 (XOUT)
- net GPIO13: now reaches U2.16 (GPIO13)
- net SWCLK: now reaches U2.24 (SWCLK)
- net SWD: now reaches U2.25 (SWD)
- net GPIO18: now reaches U2.29 (GPIO18)
- net GPIO19: now reaches U2.30 (GPIO19)
- net GPIO20: now reaches U2.31 (GPIO20)
- net GPIO21: now reaches U2.32 (GPIO21)
- net GPIO22: now reaches U2.34 (GPIO22)
- net GPIO23: now reaches U2.35 (GPIO23)
- net GPIO24: now reaches U2.36 (GPIO24)
- net GPIO25: now reaches U2.37 (GPIO25)
- net GPIO6: now reaches U2.8 (GPIO6)
- net GPIO7: now reaches U2.9 (GPIO7)
- net at R6.2, Y1.2: now also C8.1
- net at P1.A7 (D-): now also R4.1
- net at P1.A5 (CC): now also R3.1
- net at P1.A4 (VBUS), P1.A9 (VBUS), P1.B4 (VBUS)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: now also C3.1, D1.2 (A)
- net at P1.A6 (D+): now also R5.1
- net ADC0 renamed GPIO26_ADC0
- net ADC1 renamed GPIO27_ADC1
- net ADC2 renamed GPIO28_ADC2
- net ADC3 renamed GPIO29_ADC3
- net D+: no longer names the net of U2.47 (USB_DP)
- net D+: now also R5.2
- net D-: no longer names the net of U2.46 (USB_DM)
- net D-: now also R4.2
- new net VDC: D1.1 (K)
- new net XOUT: R6.1, U2.21 (XOUT)
- no-connect marks 4 -> 1
Other:
- note removed: "ITS A BLUEPRINT NO POWER OR USB CONNECTIONS ARE PRESENT"
- company: (none) -> Raspberry Pi Ltd
- title: (none) -> RP2040 Minimal Design Example
- moved on the sheet: C10, C11, C12, C13, C14, C15, C16, C4, C5, C6, C9, P1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

Commit message: 90%
Connections:
- net VDC renamed VUSB
Changed lines of the file:
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@@
 			)
 		)
-		(property "Value" "VDC"
-			(at 132.08 105.41 0)
+		(property "Value" "VUSB"
+			(at 134.62 109.2199 0)
 			(effects
 				(font
 					(size 1.27 1.27)
 				)
+				(justify left)
 			)
 		)

Commit message: RC thing PCB 95% trustworthy (six seven)
Parts:
- removed C11: 100n, Capacitor_SMD:C_0603_1608Metric_Pad1.08x0.95mm_HandSolder, symbol Device:C
- removed P1: USB_C_Plug_USB2.0, Connector_USB:USB_C_Receptacle_Molex_105450-0101, symbol Connector:USB_C_Plug_USB2.0
- removed Y1: 12Mhz, Crystal:Crystal_SMD_Abracon_ABM8G-4Pin_3.2x2.5mm, symbol Device:Crystal
- added J2: 2171790001, rctg:2171790001_MOL, symbol MainPCB_Sym_lib:2171790001
- added R6: 5.1k, Resistor_SMD:R_0603_1608Metric_Pad0.98x0.95mm_HandSolder, symbol Device:R
- added Y3: Crystal_GND24_Small, Crystal:Crystal_SMD_Abracon_ABM8G-4Pin_3.2x2.5mm, symbol Device:Crystal_GND24_Small
- R10: renamed from R7; footprint Resistor_SMD:R_0402_1005Metric -> Resistor_SMD:R_0603_1608Metric_Pad0.98x0.95mm_HandSolder
- R7: renamed from R6; footprint (none) -> Resistor_SMD:R_0603_1608Metric_Pad0.98x0.95mm_HandSolder
- R8: footprint Resistor_SMD:R_0402_1005Metric -> Resistor_SMD:R_0603_1608Metric_Pad0.98x0.95mm_HandSolder
- SW302: renamed from SW1; footprint TL3342F160QG_TR:SW_TL3342F160QG_TR -> Main_PCB:SW_TL3342F160QG_TR
- U2: footprint RP2040_minimal:RP2040-QFN-56 -> Package_DFN_QFN:QFN-56-1EP_7x7mm_P0.4mm_EP3.2x3.2mm
- U3: footprint Package_SO:SOIC-8_5.23x5.23mm_P1.27mm -> Package_SO:SOIC-8_5.3x5.3mm_P1.27mm
- renumbered C17 to C1, C12 to C10, C13 to C11, C14 to C12, C15 to C13, C16 to C14, C9 to C15, C3 to C16, C7 to C2, C8 to C3, C6 to C4, C4 to C5, C5 to C6, C10 to C8
Connections:
- net GND: now also J2.A1/B12 (GND), J2.B1/A12 (GND), R6.2, Y3.2, Y3.4
- net XIN: now also Y3.3
- net at C3.1, R7.2: now also Y3.1
- net at C16.1, D1.2 (A): now also J2.A4/B9 (VBUS), J2.B4/A9 (VBUS)
- net at R4.1: now also J2.A7 (DN1), J2.B7 (DN2)
- net at R5.1: now also J2.A6 (DP1), J2.B6 (DP2)
- net at R3.1: now also J2.B5 (CC2)
- new net: J2.A5 (CC1), R6.1
- no-connect marks 1 -> 2
Other:
- moved on the sheet: C10, C11, C12, C13, C14, C15, C16, C2, C3, D1, R3, R7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

Commit message: new RC PCB updates
Parts:
- added R9: 10k, Capacitor_SMD:C_0603_1608Metric_Pad1.08x0.95mm_HandSolder, symbol Device:R
- added SW5: TL3342F160QG_TR, Main_PCB:SW_TL3342F160QG_TR, symbol TL3342F160QG_TR:TL3342F160QG_TR
- renumbered SW302 to SW8
Connections:
- net GND: now also SW5.3
- net RUN: now also R9.1, SW5.2
- new net +3.3V: R9.2
- no-connect marks 2 -> 4
Other:
- moved on the sheet: C1, C10, C11, C12, C13, C14, C15, C16, C2, C3, C4, C5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

Commit message: G will be touched tonight
Connections:
- net +3.3V is gone; now on net +3V3: R9.2
Changed lines of the file:
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@@
 			)
 		)
-		(property "Value" "+3.3V"
+		(property "Value" "+3V3"
 			(at 158.75 131.318 0)
 			(effects

Commit message: Reviewed .sch
Parts:
- added R11, R12: 5.1k, Resistor_SMD:R_0603_1608Metric_Pad0.98x0.95mm_HandSolder, symbol Device:R
- C16: value 10u -> 4.7u
- renumbered Y3 to X1
Connections:
- net +3V3: now also R11.1, R12.1
- net GPIO0: now also R11.2
- net GPIO1: now also R12.2
Other:
- moved on the sheet: R3, R6, R9, SW5

Commit message: Final touches
Parts:
- renumbered C5 to C1, C13 to C10, C14 to C11, C15 to C12, C1 to C13, C16 to C14, C6 to C2, C4 to C3, C2 to C4, C3 to C5, C8 to C6, C10 to C7, C11 to C8, C12 to C9, R9 to R1, R8 to R10, R7 to R2, R11 to R3, R12 to R4, R6 to R5, R4 to R6, R5 to R7, R3 to R8, R10 to R9, SW5 to SW4, SW8 to SW5
