File: Hardware/Main_PCB/connections.kicad_sch (KiCad schematic)
At the start: 6 parts, among them J601 Conn_01x08_Pin, J602 Conn_01x03_Pin, J603 Servo con, U601 NRF24L01, U602 SN74LV1T34DBV

Commit message: Finished MainPCB v3
Parts:
- added TP601: +VPROT test point, TestPoint:TestPoint_Pad_D1.0mm, symbol Connector:TestPoint
Connections:
- net VDC renamed +VPROT
- net +VPROT: now also TP601.1
Changed lines of the file:
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@@
 	(paper "A5")
 	(rectangle
-		(start 21.59 21.59)
+		(start 21.59 17.526)
 		(end 92.71 48.26)
 		(stroke
@@
 	(text "Connectors for ESC/BMS-board"
 		(exclude_from_sim no)
-		(at 44.196 24.13 0)
+		(at 44.196 20.32 0)
 		(effects
 			(font
@@
 		)
 	)
+	(junction
+		(at 66.04 29.21)
+		(diameter 0)
+		(color 0 0 0 0)
+	)
 	(no_connect
 		(at 34.29 45.72)
@@
 	(wire
 		(pts
-			(xy 66.04 33.02) (xy 66.04 31.75)
+			(xy 66.04 27.94) (xy 66.04 29.21)
 		)
 		(stroke
@@
 	(wire
 		(pts
-			(xy 67.31 35.56) (xy 59.69 35.56)
+			(xy 67.31 35.56) (xy 58.42 35.56)
 		)
 		(stroke
@@
 	(wire
 		(pts
-			(xy 59.69 35.56) (xy 59.69 31.75)
+			(xy 66.04 29.21) (xy 66.04 33.02)
+		)
+		(stroke
+			(width 0)
+			(type default)
+		)
+	)
+	(wire
+		(pts
+			(xy 66.04 29.21) (xy 71.12 29.21)
+		)
+		(stroke
+			(width 0)
+			(type default)
+		)
+	)
+	(wire
+		(pts
+			(xy 58.42 35.56) (xy 58.42 27.94)
 		)
 		(stroke
@@
 	(symbol
 		(lib_id "power:VDC")
-		(at 66.04 31.75 0)
+		(at 66.04 27.94 0)
 		(unit 1)
 		(exclude_from_sim no)
@@
 		(dnp no)
 		(property "Reference" "#PWR0604"
-			(at 66.04 35.56 0)
-			(effects
-				(font
-					(size 1.27 1.27)
-				)
-				(hide yes)
-			)
-		)
-		(property "Value" "VDC"
-			(at 66.04 28.194 0)
+			(at 66.04 31.75 0)
+			(effects
+				(font
+					(size 1.27 1.27)
+				)
+				(hide yes)
+			)
+		)
+		(property "Value" "+VPROT"
+			(at 66.04 24.384 0)
 			(effects
 				(font
@@
 		)
 		(property "Footprint" ""
-			(at 66.04 31.75 0)
+			(at 66.04 27.94 0)
 			(effects
 				(font
@@
 		)
 		(property "Datasheet" ""
-			(at 66.04 31.75 0)
+			(at 66.04 27.94 0)
 			(effects
 				(font
@@
 		)
 		(property "Description" "Power symbol creates a global label with name \"VDC\""
-			(at 66.04 31.75 0)
+			(at 66.04 27.94 0)
 			(effects
 				(font
@@
 	(symbol
 		(lib_id "power:+3.3V")
-		(at 59.69 31.75 0)
+		(at 58.42 27.94 0)
 		(unit 1)
 		(exclude_from_sim no)
@@
 		(dnp no)
 		(property "Reference" "#PWR0603"
-			(at 59.69 35.56 0)
+			(at 58.42 31.75 0)
 			(effects
 				(font
@@
 		)
 		(property "Value" "+3.3V"
-			(at 59.69 28.194 0)
+			(at 58.42 24.384 0)
 			(effects
 				(font
@@
 		)
 		(property "Footprint" ""
-			(at 59.69 31.75 0)
+			(at 58.42 27.94 0)
 			(effects
 				(font
@@
 		)
 		(property "Datasheet" ""
-			(at 59.69 31.75 0)
+			(at 58.42 27.94 0)
 			(effects
 				(font
@@
 		)
 		(property "Description" "Power symbol creates a global label with name \"+3.3V\""
-			(at 59.69 31.75 0)
+			(at 58.42 27.94 0)
 			(effects
 				(font
@@
 					(unit 1)
 				)
+			)
+		)
+	)
+	(symbol
+		(lib_id "Connector:TestPoint")
+		(at 71.12 29.21 270)
+		(unit 1)
+		(exclude_from_sim no)
+		(in_bom yes)
+		(on_board yes)
+		(dnp no)
+		(property "Reference" "TP601"
+			(at 76.2 27.9399 90)
+			(effects
+				(font
+					(size 1.27 1.27)
+				)
+				(justify left)
+			)
+		)
+		(property "Value" "+VPROT test point"
+			(at 73.152 30.988 90)
+			(effects
+				(font
+					(size 1.27 1.27)
+				)
+				(justify left)
+			)
+		)
+		(property "Footprint" "TestPoint:TestPoint_Pad_D1.0mm"
+			(at 71.12 34.29 0)
+			(effects
+				(font
+					(size 1.27 1.27)
+				)
+				(hide yes)
+			)
+		)
+		(property "Datasheet" "~"
+			(at 71.12 34.29 0)
+			(effects
+				(font
+					(size 1.27 1.27)
+				)
+				(hide yes)
+			)
+		)
+		(property "Description" "test point"
+			(at 71.12 29.21 0)
+			(effects
+				(font
+					(size 1.27 1.27)
+				)
+				(hide yes)
+			)
+		)
+		(pin "1"
+		)
+		(instances
+			(project ""
+				(path "/90d7beec-e1a2-46f8-bbb2-6b8f3489db10/2fd609f6-122d-440e-b3d6-5f283f47ac3b"
+					(reference "TP601")
+					(unit 1)
+				)

Commit message: Beautifying the Master Controller
Other:
- company: (none) -> Made by Liubomir Stanev
- title: (none) -> Master controller
Changed lines of the file:
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@@
 	(generator_version "9.0")
 	(paper "A5")
+	(title_block
+		(title "Master controller")
+		(date "22/12/2025")
+		(company "Made by Liubomir Stanev")
+		(comment 1 "Page 6: Connectors")
+	)
 	(rectangle
 		(start 21.59 17.526)
@@
 			)
 		)
-		(property "Datasheet" "http://www.nordicsemi.com/eng/content/download/2730/34105/file/nRF24L01_Product_Specification_v2_0.pdf"
+		(property "Datasheet" "https://www.handsontec.com/dataspecs/module/NRF24L01+PA.pdf"
 			(at 44.45 97.79 0)
 			(effects
