File: Hardware/Main_PCB/rp2040.kicad_sch (KiCad schematic)
At the start: 29 parts, among them J301 2171790001, SW301 TL3342F160QG_TR, SW302 TL3342F160QG_TR, U301 RP2040, U302 W25Q128JVS, Y301 12Mhz

Commit message: V1.1 of the MainPCB
Parts:
- removed Y301: 12Mhz, Crystal:Crystal_SMD_Abracon_ABM8G-4Pin_3.2x2.5mm, symbol Device:Crystal
- added R301: 10k, Capacitor_SMD:C_0603_1608Metric_Pad1.08x0.95mm_HandSolder, symbol Device:R
- added Y301: 12MHz, Crystal:Crystal_SMD_Abracon_ABM8G-4Pin_3.2x2.5mm, symbol Device:Crystal_GND24
- renumbered R301 to R302, R302 to R303, R303 to R304, R304 to R305, R305 to R306, R306 to R307, R307 to R308
Connections:
- net +3.3V: now also R301.2
- net GND: now also Y301.2, Y301.4
- net RUN: now also R301.1
- net XIN: now also Y301.1
- net at C305.1, R302.2: now also Y301.3
- net Data-: now reaches J301.A7 (DN1), J301.B7 (DN2), R305.1
- net Data+: now reaches J301.A6 (DP1), J301.B6 (DP2), R304.1

Commit message: Finished MainPCB v3
Connections:
- net VDC renamed +VPROT
Changed lines of the file:
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@@
 	(wire
 		(pts
-			(xy 237.49 101.6) (xy 237.49 100.33)
+			(xy 234.95 101.6) (xy 234.95 100.33)
 		)
 		(stroke
@@
 	(wire
 		(pts
-			(xy 240.03 101.6) (xy 237.49 101.6)
+			(xy 240.03 101.6) (xy 234.95 101.6)
 		)
 		(stroke
@@
 	(symbol
 		(lib_id "power:VDC")
-		(at 237.49 100.33 0)
+		(at 234.95 100.33 0)
 		(unit 1)
 		(exclude_from_sim no)
@@
 		(on_board yes)
 		(dnp no)
-		(fields_autoplaced yes)
 		(property "Reference" "#PWR0317"
-			(at 237.49 104.14 0)
+			(at 234.95 104.14 0)
 			(effects
 				(font
@@
 			)
 		)
-		(property "Value" "VDC"
-			(at 237.49 95.25 0)
+		(property "Value" "+VPROT"
+			(at 230.886 96.774 0)
 			(effects
 				(font
 					(size 1.27 1.27)
 				)
+				(justify left)
 			)
 		)
 		(property "Footprint" ""
-			(at 237.49 100.33 0)
+			(at 234.95 100.33 0)
 			(effects
 				(font
@@
 		)
 		(property "Datasheet" ""
-			(at 237.49 100.33 0)
+			(at 234.95 100.33 0)
 			(effects
 				(font
@@
 		)
 		(property "Description" "Power symbol creates a global label with name \"VDC\""
-			(at 237.49 100.33 0)
+			(at 234.95 100.33 0)
 			(effects
 				(font

Commit message: Footprint updated
Parts:
- J301: footprint MainPCB:2171790001_MOL -> SPRO3:2171790001_MOL
Other:
- moved on the sheet: R303, R304, R305, R306
Changed lines of the file:
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@@
 	(wire
 		(pts
-			(xy 185.42 110.49) (xy 180.34 110.49)
+			(xy 184.15 111.76) (xy 182.88 111.76)
 		)
 		(stroke
@@
 	(wire
 		(pts
-			(xy 201.93 110.49) (xy 193.04 110.49)
+			(xy 201.93 111.76) (xy 191.77 111.76)
 		)
 		(stroke
@@
 	(wire
 		(pts
-			(xy 139.7 100.33) (xy 170.18 100.33)
+			(xy 139.7 100.33) (xy 168.91 100.33)
 		)
 		(stroke
@@
 	(wire
 		(pts
-			(xy 170.18 119.38) (xy 185.42 119.38)
+			(xy 168.91 119.38) (xy 184.15 119.38)
 		)
 		(stroke
@@
 	(wire
 		(pts
-			(xy 193.04 119.38) (xy 200.66 119.38)
+			(xy 191.77 119.38) (xy 200.66 119.38)
 		)
 		(stroke
@@
 	(wire
 		(pts
-			(xy 201.93 116.84) (xy 201.93 110.49)
+			(xy 201.93 116.84) (xy 201.93 111.76)
 		)
 		(stroke
@@
 	(wire
 		(pts
-			(xy 185.42 140.97) (xy 180.34 140.97)
+			(xy 184.15 134.62) (xy 182.88 134.62)
 		)
 		(stroke
@@
 	(wire
 		(pts
-			(xy 180.34 110.49) (xy 180.34 111.76)
+			(xy 182.88 111.76) (xy 182.88 113.03)
 		)
 		(stroke
@@
 	(wire
 		(pts
-			(xy 167.64 127) (xy 167.64 102.87)
+			(xy 166.37 127) (xy 166.37 102.87)
 		)
 		(stroke
@@
 	(wire
 		(pts
-			(xy 180.34 140.97) (xy 180.34 142.24)
+			(xy 182.88 134.62) (xy 182.88 135.89)
 		)
 		(stroke
@@
 	(wire
 		(pts
-			(xy 193.04 127) (xy 194.31 127)
+			(xy 191.77 127) (xy 194.31 127)
 		)
 		(stroke
@@
 	(wire
 		(pts
-			(xy 139.7 102.87) (xy 167.64 102.87)
+			(xy 139.7 102.87) (xy 166.37 102.87)
 		)
 		(stroke
@@
 	(wire
 		(pts
-			(xy 198.12 127) (xy 198.12 140.97)
+			(xy 198.12 127) (xy 198.12 134.62)
 		)
 		(stroke
@@
 	(wire
 		(pts
-			(xy 170.18 100.33) (xy 170.18 119.38)
+			(xy 168.91 100.33) (xy 168.91 119.38)
 		)
 		(stroke
@@
 	(wire
 		(pts
-			(xy 167.64 127) (xy 185.42 127)
+			(xy 166.37 127) (xy 184.15 127)
 		)
 		(stroke
@@
 	(wire
 		(pts
-			(xy 193.04 140.97) (xy 198.12 140.97)
+			(xy 191.77 134.62) (xy 198.12 134.62)
 		)
 		(stroke
@@
 	(symbol
 		(lib_id "Device:R")
-		(at 189.23 127 270)
+		(at 187.96 127 270)
 		(mirror x)
 		(unit 1)
@@
 		(dnp no)
 		(property "Reference" "R305"
-			(at 189.23 124.46 90)
+			(at 187.96 124.46 90)
 			(effects
 				(font
@@
 		)
 		(property "Value" "27"
-			(at 189.23 129.54 90)
+			(at 187.96 129.54 90)
 			(effects
 				(font
@@
 		)
 		(property "Footprint" "Resistor_SMD:R_0603_1608Metric_Pad0.98x0.95mm_HandSolder"
-			(at 189.23 128.778 90)
+			(at 187.96 128.778 90)
 			(effects
 				(font
@@
 		)
 		(property "Datasheet" "~"
-			(at 189.23 127 0)
+			(at 187.96 127 0)
 			(effects
 				(font
@@
 		)
 		(property "Description" "Resistor"
-			(at 189.23 127 0)
+			(at 187.96 127 0)
 			(effects
 				(font
@@
 			)
 		)
-		(property "Footprint" "MainPCB:2171790001_MOL"
+		(property "Footprint" "SPRO3:2171790001_MOL"
 			(at 203.2 116.84 0)
 			(effects
@@
 	(symbol
 		(lib_id "power:GND")
-		(at 180.34 142.24 0)
+		(at 182.88 135.89 0)
 		(mirror y)
 		(unit 1)
@@
 		(dnp no)
 		(property "Reference" "#PWR0315"
-			(at 180.34 148.59 0)
+			(at 182.88 142.24 0)
 			(effects
 				(font
@@
 		)
 		(property "Value" "GND"
-			(at 180.34 146.05 0)
+			(at 182.88 139.7 0)
 			(effects
 				(font
@@
 		)
 		(property "Footprint" ""
-			(at 180.34 142.24 0)
+			(at 182.88 135.89 0)
 			(effects
 				(font
@@
 		)
 		(property "Datasheet" ""
-			(at 180.34 142.24 0)
+			(at 182.88 135.89 0)
 			(effects
 				(font
@@
 		)
 		(property "Description" ""
-			(at 180.34 142.24 0)
+			(at 182.88 135.89 0)
 			(effects
 				(font
@@
 	(symbol
 		(lib_id "power:GND")
-		(at 180.34 111.76 0)
+		(at 182.88 113.03 0)
 		(mirror y)
 		(unit 1)
@@
 		(dnp no)
 		(property "Reference" "#PWR0314"
-			(at 180.34 118.11 0)
+			(at 182.88 119.38 0)
 			(effects
 				(font
@@
 		)
 		(property "Value" "GND"
-			(at 180.34 115.57 0)
+			(at 182.88 116.84 0)
 			(effects
 				(font
@@
 		)
 		(property "Footprint" ""
-			(at 180.34 111.76 0)
+			(at 182.88 113.03 0)
 			(effects
 				(font
@@
 		)
 		(property "Datasheet" ""
-			(at 180.34 111.76 0)
+			(at 182.88 113.03 0)
 			(effects
 				(font
@@
 		)
 		(property "Description" ""
-			(at 180.34 111.76 0)
+			(at 182.88 113.03 0)
 			(effects
 				(font
@@
 	(symbol
 		(lib_id "Device:R")
-		(at 189.23 140.97 270)
+		(at 187.96 134.62 270)
 		(mirror x)
 		(unit 1)
@@
 		(dnp no)
 		(property "Reference" "R306"
-			(at 189.23 138.684 90)
+			(at 187.96 132.334 90)
 			(effects
 				(font
@@
 		)
 		(property "Value" "5.1k"
-			(at 188.976 143.256 90)
+			(at 187.706 136.906 90)
 			(effects
 				(font
@@
 		)
 		(property "Footprint" "Resistor_SMD:R_0603_1608Metric_Pad0.98x0.95mm_HandSolder"
-			(at 189.23 142.748 90)
+			(at 187.96 136.398 90)
 			(effects
 				(font
@@
 		)
 		(property "Datasheet" "~"
-			(at 189.23 140.97 0)
+			(at 187.96 134.62 0)
 			(effects
 				(font
@@
 		)
 		(property "Description" "Resistor"
-			(at 189.23 140.97 0)
+			(at 187.96 134.62 0)
 			(effects
 				(font
@@
 	(symbol
 		(lib_id "Device:R")
-		(at 189.23 110.49 270)
+		(at 187.96 111.76 270)
 		(mirror x)
 		(unit 1)
@@
 		(dnp no)
 		(property "Reference" "R303"
-			(at 189.23 108.204 90)
+			(at 187.96 109.474 90)
 			(effects
 				(font
@@
 		)
 		(property "Value" "5.1k"
-			(at 188.976 112.776 90)
+			(at 187.706 114.046 90)
 			(effects
 				(font
@@
 		)
 		(property "Footprint" "Resistor_SMD:R_0603_1608Metric_Pad0.98x0.95mm_HandSolder"
-			(at 189.23 112.268 90)
+			(at 187.96 113.538 90)
 			(effects
 				(font
@@
 		)
 		(property "Datasheet" "~"
-			(at 189.23 110.49 0)
+			(at 187.96 111.76 0)
 			(effects
 				(font
@@
 		)
 		(property "Description" "Resistor"
-			(at 189.23 110.49 0)
+			(at 187.96 111.76 0)
 			(effects
 				(font
@@
 	(symbol
 		(lib_id "Device:R")
-		(at 189.23 119.38 270)
+		(at 187.96 119.38 270)
 		(mirror x)
 		(unit 1)
@@
 		(dnp no)
 		(property "Reference" "R304"
-			(at 189.23 116.84 90)
+			(at 187.96 116.84 90)
 			(effects
 				(font
@@
 		)
 		(property "Value" "27"
-			(at 189.23 121.92 90)
+			(at 187.96 121.92 90)
 			(effects
 				(font
@@
 		)
 		(property "Footprint" "Resistor_SMD:R_0603_1608Metric_Pad0.98x0.95mm_HandSolder"
-			(at 189.23 121.158 90)
+			(at 187.96 121.158 90)
 			(effects
 				(font
@@
 		)
 		(property "Datasheet" "~"
-			(at 189.23 119.38 0)
+			(at 187.96 119.38 0)
 			(effects
 				(font
@@
 		)
 		(property "Description" "Resistor"
-			(at 189.23 119.38 0)
+			(at 187.96 119.38 0)
 			(effects
 				(font

Commit message: Beautifying the Master Controller
Other:
- company: (none) -> Made by Liubomir Stanev
- title: (none) -> Master controller
Changed lines of the file:
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@@
 	(generator_version "9.0")
 	(paper "A3")
+	(title_block
+		(title "Master controller")
+		(date "22/12/2025")
+		(company "Made by Liubomir Stanev")
+		(comment 1 "Page 3: Microcontroller")
+	)
 	(text "Flash"
 		(exclude_from_sim no)
