File: Hardware/Main_PCB/sonar.kicad_sch (KiCad schematic)
At the start: 13 parts, among them J201 Sonar, U201 TUSS4470TRTJT

Commit message: Beautifying the Master Controller
Other:
- company: (none) -> Made by Liubomir Stanev
- title: (none) -> Master controller
Changed lines of the file:
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@@
 	(generator_version "9.0")
 	(paper "A5")
+	(title_block
+		(title "Master controller")
+		(date "22/12/2025")
+		(company "Made by Liubomir Stanev")
+		(comment 1 "Page 2: SONAR")
+	)
 	(text "40V"
 		(exclude_from_sim no)
